File: kicad/clock.kicad_sch (KiCad schematic)
At the start: 59 parts, among them J1 USB_C_Receptacle_PowerOnly_6P, J2 USB_A, J5 Barrel_Jack, SW1 SW_SPDT, SW2 SW_Push, SW3 SW_Push, U1 4511, U10 4060, U11 4013, U18 4081, U2 4511, U20 FJS18101APG, U21 FJS18101APG, U22 FJS18101APG, U23 FJS18101APG, U24 FJS18101APG, U25 FJS18101APG, U3 4511, U4 4511, U5 4511, U6 4511, U7 4518, U8 4518, U9 4518, Y1 32768

Commit message: Completed article
Parts:
- added H5, H6: MountingHole, MountingHole:MountingHole_3.5mm, symbol Mechanical:MountingHole
Other:
- title: Logic Clock -> Large Logic Clock
- moved on the sheet: H1, H2
Changed lines of the file:
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@@
 	(paper "A3")
 	(title_block
-		(title "Logic Clock")
-		(date "2025-10-31")
-		(rev "1.0")
+		(title "Large Logic Clock")
+		(date "2025-12-12")
+		(rev "3.0")
 	)
 	(text "Unused Device"
@@
 	)
 	(symbol
+		(lib_id "Mechanical:MountingHole")
+		(at 224.79 275.59 0)
+		(unit 1)
+		(exclude_from_sim no)
+		(in_bom yes)
+		(on_board yes)
+		(dnp no)
+		(fields_autoplaced yes)
+		(property "Reference" "H5"
+			(at 227.33 274.32 0)
+			(effects
+				(font
+					(size 1.27 1.27)
+				)
+				(justify left)
+			)
+		)
+		(property "Value" "MountingHole"
+			(at 227.33 276.86 0)
+			(effects
+				(font
+					(size 1.27 1.27)
+				)
+				(justify left)
+			)
+		)
+		(property "Footprint" "MountingHole:MountingHole_3.5mm"
+			(at 224.79 275.59 0)
+			(effects
+				(font
+					(size 1.27 1.27)
+				)
+				(hide yes)
+			)
+		)
+		(property "Datasheet" "~"
+			(at 224.79 275.59 0)
+			(effects
+				(font
+					(size 1.27 1.27)
+				)
+				(hide yes)
+			)
+		)
+		(property "Description" "Mounting Hole without connection"
+			(at 224.79 275.59 0)
+			(effects
+				(font
+					(size 1.27 1.27)
+				)
+				(hide yes)
+			)
+		)
+		(instances
+			(project "clock"
+				(path "/52556f3a-6d57-4670-ba4a-28f0dc053e76"
+					(reference "H5")
+					(unit 1)
+				)
+			)
+		)
+	)
+	(symbol
 		(lib_id "4xxx:4060")
 		(at 248.92 200.66 0)
@@
 	(symbol
 		(lib_id "Mechanical:MountingHole")
-		(at 248.92 251.46 0)
+		(at 248.92 252.73 0)
 		(unit 1)
 		(exclude_from_sim no)
@@
 		(fields_autoplaced yes)
 		(property "Reference" "H2"
-			(at 251.46 250.19 0)
+			(at 251.46 251.46 0)
 			(effects
 				(font
@@
 		)
 		(property "Value" "MountingHole"
-			(at 251.46 252.73 0)
+			(at 251.46 254 0)
 			(effects
 				(font
@@
 		)
 		(property "Footprint" "MountingHole:MountingHole_3.5mm"
-			(at 248.92 251.46 0)
+			(at 248.92 252.73 0)
 			(effects
 				(font
@@
 		)
 		(property "Datasheet" "~"
-			(at 248.92 251.46 0)
+			(at 248.92 252.73 0)
 			(effects
 				(font
@@
 		)
 		(property "Description" "Mounting Hole without connection"
-			(at 248.92 251.46 0)
+			(at 248.92 252.73 0)
 			(effects
 				(font
@@
 	(symbol
 		(lib_id "Mechanical:MountingHole")
-		(at 224.79 251.46 0)
+		(at 224.79 252.73 0)
 		(unit 1)
 		(exclude_from_sim no)
@@
 		(fields_autoplaced yes)
 		(property "Reference" "H1"
-			(at 227.33 250.19 0)
+			(at 227.33 251.46 0)
 			(effects
 				(font
@@
 		)
 		(property "Value" "MountingHole"
-			(at 227.33 252.73 0)
+			(at 227.33 254 0)
 			(effects
 				(font
@@
 		)
 		(property "Footprint" "MountingHole:MountingHole_3.5mm"
-			(at 224.79 251.46 0)
+			(at 224.79 252.73 0)
 			(effects
 				(font
@@
 		)
 		(property "Datasheet" "~"
-			(at 224.79 251.46 0)
+			(at 224.79 252.73 0)
 			(effects
 				(font
@@
 		)
 		(property "Description" "Mounting Hole without connection"
-			(at 224.79 251.46 0)
+			(at 224.79 252.73 0)
 			(effects
 				(font
@@
 					(unit 1)
 				)
+			)
+		)
+	)
+	(symbol
+		(lib_id "Mechanical:MountingHole")
+		(at 248.92 275.59 0)
+		(unit 1)
+		(exclude_from_sim no)
+		(in_bom yes)
+		(on_board yes)
+		(dnp no)
+		(fields_autoplaced yes)
+		(property "Reference" "H6"
+			(at 251.46 274.32 0)
+			(effects
+				(font
+					(size 1.27 1.27)
+				)
+				(justify left)
+			)
+		)
+		(property "Value" "MountingHole"
+			(at 251.46 276.86 0)
+			(effects
+				(font
+					(size 1.27 1.27)
+				)
+				(justify left)
+			)
+		)
+		(property "Footprint" "MountingHole:MountingHole_3.5mm"
+			(at 248.92 275.59 0)
+			(effects
+				(font
+					(size 1.27 1.27)
+				)
+				(hide yes)
+			)
+		)
+		(property "Datasheet" "~"
+			(at 248.92 275.59 0)
+			(effects
+				(font
+					(size 1.27 1.27)
+				)
+				(hide yes)
+			)
+		)
+		(property "Description" "Mounting Hole without connection"
+			(at 248.92 275.59 0)
+			(effects
+				(font
+					(size 1.27 1.27)
+				)
+				(hide yes)
+			)
+		)
+		(instances
+			(project "clock"
+				(path "/52556f3a-6d57-4670-ba4a-28f0dc053e76"
+					(reference "H6")
+					(unit 1)
+				)
